File: hardware/head/head.kicad_sch (KiCad schematic)
At the start: 50 parts, among them J1 Head bundle, J10 CM4 socket 101-200, J2 ToF, J3 I2C breakout, J4 Eye LED, J5 Speaker, J6 Fan, J7 Microphone, J8 Camera, J9 CM4 socket 1-100, Q1 AO3400A, U2 LMR51635XDDCR, U3 AMS1117-3.3, U4 MAX98357AETE+T, U5 BMI088 module

Commit message: Head carrier PCB: BMI088 on board, fallbacks, 1.1 MHz buck (one connection open)
BMI088 chip in place of the module, with links to cut for an external
module on J3; a wide 3 A link (JP1) between the buck and the 5 V rail
with external 5 V pads (J12); a link (JP3) in the amplifier's 5 V with
module pads (J11). Buck now LMR51635YDDCR with a 4.7 uH SWPA6045.
Silkscreen labels and the name block on the back. ToF and eye headers
moved 0.3 mm clear of the module's edge. One I2C SCL connection still
open; fab outputs not regenerated. See docs/head-pcb.md 9.3.
Parts:
- removed R5: 100R, Resistor_SMD:R_0603_1608Metric, symbol Device:R
- removed R7: 330R, Resistor_SMD:R_0603_1608Metric, symbol Device:R
- removed U5: BMI088 module, DukkiHead:BMI088_Module, symbol DukkiHead:BMI088_Module
- added C15, C16: 100n 50V, Capacitor_SMD:C_0603_1608Metric, symbol Device:C
- added J11: Ext amp, Connector_PinHeader_2.54mm:PinHeader_1x07_P2.54mm_Vertical, symbol Connector_Generic:Conn_01x07
- added J12: Ext 5V, Connector_PinHeader_2.54mm:PinHeader_1x04_P2.54mm_Vertical, symbol Connector_Generic:Conn_01x04
- added J4: Eye LED, Connector_JST:JST_PH_B3B-PH-K_1x03_P2.00mm_Vertical, symbol Connector_Generic:Conn_01x03
- added JP1: cut for ext 5V, DukkiHead:SolderJumper-2_Wide_Bridged_3A, symbol Jumper:SolderJumper_2_Bridged
- added JP3: cut for ext amp, DukkiHead:SolderJumper-2_Wide_Bridged_3A, symbol Jumper:SolderJumper_2_Bridged
- added JP4, JP5: cut for ext IMU, Jumper:SolderJumper-2_P1.3mm_Bridged_RoundedPad1.0x1.5mm, symbol Jumper:SolderJumper_2_Bridged
- added R6: 100k, Resistor_SMD:R_0603_1608Metric, symbol Device:R
- added U5: BMI088, Package_LGA:Bosch_LGA-16_4.5x3mm_P0.5mm_LayoutBorder7x1y_ClockwisePinNumbering, symbol DukkiHead:BMI088
- L1: value 10u -> 4.7u; footprint Inductor_SMD:L_Sunlord_MWSA0603S -> Inductor_SMD:L_Sunlord_SWPA6045S; LCSC C132141 -> C78804; MPN Sunlord MWSA0603S-100MT, 10 uH, 5.5 A saturation -> Sunlord SWPA6045S4R7MT, 4.7 uH, 5.5 A saturation
- R5: renamed from R6; value 100k -> 100R; LCSC C25803 -> C22775
- R7: renamed from J4; value Eye LED -> 330R; footprint Connector_JST:JST_PH_B3B-PH-K_1x03_P2.00mm_Vertical -> Resistor_SMD:R_0603_1608Metric; symbol Connector_Generic:Conn_01x03 -> Device:R; LCSC (none) -> C23138; MPN JST B3B-PH-K-S, through hole, fitted by hand -> (none); now in the parts list
- R8, R9: now fitted
- U2: value LMR51635XDDCR -> LMR51635YDDCR; LCSC C42432812 -> C45262770
Connections:
- net +3V3: now also C15.1, C16.1, U5.10 (SDO2), U5.11 (VDDIO), U5.14 (~{CSB1}), U5.15 (SDO1), U5.3 (VDD), U5.7 (PS)
- net +5V: now also J11.7 (Pin_7), J12.3 (Pin_3), J4.1 (Pin_1), JP1.2 (B), JP3.1 (A); no longer C12.1, C13.1, C6.1, C7.1, C8.1, L1.2, R1.1, R3.1, R7.1 (Pin_1), U4.7 (VDD), U4.8 (VDD)
- net EYE_DATA: now also R7.1
- net EYE_DIN: now also J4.2 (Pin_2)
- net FAN_G: now also R5.2, R6.1; no longer R5.1
- net FAN_PWM: now also R5.1
- net GND: now also C15.2, C16.2, J11.6 (Pin_6), J12.2 (Pin_2), J12.4 (Pin_4), J4.3 (Pin_3), R6.2, U5.2 (GNDA), U5.4 (GNDA), U5.6 (GNDIO); no longer R5.2, R7.3 (Pin_3)
- net I2C8_SCL: now also JP5.1 (A)
- net I2C8_SDA: now also JP4.1 (A)
- net SAI2_LRCK: now also J11.1 (Pin_1)
- net SAI2_SCLK: now also J11.2 (Pin_2)
- net SAI2_SDO: now also J11.3 (Pin_3)
- net VBAT_IN: now also J12.1 (Pin_1)
- new net 5V_BUCK: C6.1, C7.1, C8.1, JP1.1 (A), L1.2, R1.1
- new net AMP_5V: C12.1, C13.1, JP3.2 (B), R3.1, U4.7 (VDD), U4.8 (VDD)
- new net IMU_SCL: JP5.2 (B), U5.8 (SCK/SCL)
- new net IMU_SDA: JP4.2 (B), U5.9 (SDI/SDA)
- no-connect marks 133 -> 134
Other:
- note added: "BMI088 on the board, I2C: PS and CSB1 high, CSB2 open (allowed in I2C mode); SDO1 and SDO2 high: accelerometer 0x19, gyroscope 0x69 (strapped so the pin rows need no vias between alternate pins). R8, R9: the bus pull-ups (the ToF breakout adds 10k). Cut JP4 and JP5 to use an external IMU module on J3"
- note added: "C15 at VDD, C16 at VDDIO"
- note added: "External fallbacks"
- note added: "J11: LRC, BCLK, DIN, GAIN (open), SD (open: module's own pull-up), GND, Vin"
- note added: "J12: 1 B+ out, 2 GND, 3 5V in, 4 GND"
- note added: "LMR51635Y, 1.1 MHz, 4.7 uH (TI table 8-2: 3.3 uH). 82k/15k sets 5.17 V. EN tied to VIN. F6 (2 A) on the bridge fuses this feed. JP1 joins the buck to the 5 V rail: cut it to feed 5 V from outside (J12). The feedback divider stays on the buck side"
- note added: "MAX98357A on SAI2. SD_MODE 1M to 5 V: (L+R)/2 mono. GAIN open = 9 dB; fit R4 (100k to GND) for 15 dB. JP3 feeds it: cut JP3 to use an external amplifier module on J11"
- note added: "Spare I2C8, same order; external IMU module here"
- note added: "Wire pads, 2.54 mm. J12: cut JP1 and feed 5 V from an external step-down. J11: cut JP3 and wire an amplifier module, pins in the generic module's order. J3 (section 6) takes an external IMU module"
- note removed: "LMR51635X, 400 kHz, TI table 8-2 values. 82k/15k sets 5.17 V. EN tied to VIN. F6 (2 A) on the bridge fuses this feed"
- note removed: "MAX98357A on SAI2. SD_MODE 1M to 5 V: (L+R)/2 mono. GAIN open = 9 dB; fit R4 (100k to GND) for 15 dB"
- note removed: "Pull-ups on the modules (ToF 10k, BMI088 3.3k): R8, R9 not fitted. BMI088 SDO to GND: 0x18 and 0x68"
- note removed: "Spare I2C8, same order"
- moved on the sheet: R5

Commit message: Head carrier PCB: SPI breakout pads (SPI2 M1) on the bottom
J13: nine wire pads under the module along the top edge (GND, 5V,
3V3, MOSI, MISO, CLK, CS0, INT, spare GPIO) on SPI2 M1, the RK3576 SPI
the eye LED leaves free, plus GPIO6 and GPIO5. The board is routed
again from placement with J13 in it; new scripts/kicad/sync_head_pcb.py
syncs a routed board with its schematic. The maze router now keeps
holes and footprint keep-outs clear, sees jumper bridges and uses
per-net clearances; the tidy gains an undangle stage and stitches
floating pour. DRC 0 violations; two module ground pins (J9 32, 33)
are boxed in and left unconnected, documented in docs/head-pcb.md 6.2.
Parts:
- added J13: SPI pads, DukkiHead:SolderPads_1x09_P2.54mm_SPI, symbol Connector_Generic:Conn_01x09
Connections:
- net +3V3: now also J13.3 (Pin_3)
- net +5V: now also J13.2 (Pin_2)
- net GND: now also J13.1 (Pin_1)
- net SPI2_MOSI: now reaches J9.28 (GPIO13)
- net SPI2_MOSI: now also J13.4 (Pin_4)
- net SPI_INT: now reaches J9.30 (GPIO6)
- net SPI_INT: now also J13.8 (Pin_8)
- net SPI2_CLK: now reaches J9.31 (GPIO12)
- net SPI2_CLK: now also J13.6 (Pin_6)
- net SPI_IO: now reaches J9.34 (GPIO5)
- net SPI_IO: now also J13.9 (Pin_9)
- net SPI2_MISO: now reaches J9.46 (GPIO22)
- net SPI2_MISO: now also J13.5 (Pin_5)
- net SPI2_CS0: now reaches J9.54 (GPIO4)
- net SPI2_CS0: now also J13.7 (Pin_7)
- no-connect marks 134 -> 128
Other:
- note added: "J13: 1 GND, 2 5V, 3 3V3, 4 MOSI, 5 MISO, 6 CLK, 7 CS0, 8 INT, 9 spare GPIO"
- note added: "SPI breakout"
- note added: "SPI2 M1 for a future SPI device, untested. Wire pads on the bottom, under the module, along the top edge. CLK GPIO12 (CM4 31), MOSI GPIO13 (28), MISO GPIO22 (46), CS0 GPIO4 (54), INT GPIO6 (30), spare GPIO5 (34)"
Changed lines of the file:
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@@
   (label "SAI2_SDI" (at 88.9 73.66 0) (fields_autoplaced yes)
     (effects (font (size 1.27 1.27)) (justify left bottom)))
-  (no_connect (at 27.94 73.66))
+  (label "SPI2_MOSI" (at 27.94 73.66 180) (fields_autoplaced yes)
+    (effects (font (size 1.27 1.27)) (justify right bottom)))
   (no_connect (at 88.9 76.2))
-  (no_connect (at 27.94 76.2))
-  (no_connect (at 88.9 78.74))
+  (label "SPI_INT" (at 27.94 76.2 180) (fields_autoplaced yes)
+    (effects (font (size 1.27 1.27)) (justify right bottom)))
+  (label "SPI2_CLK" (at 88.9 78.74 0) (fields_autoplaced yes)
+    (effects (font (size 1.27 1.27)) (justify left bottom)))
   (symbol (lib_id "power:GND") (at 27.94 78.74 270) (unit 1)
     (exclude_from_sim no) (in_bom no) (on_board yes) (dnp no)
@@
     (instances (project "head" (path "/a08b5940-33cf-5ae8-8123-d7cbee5060cd" (reference "#PWR010") (unit 1))))
   )
-  (no_connect (at 27.94 81.28))
+  (label "SPI_IO" (at 27.94 81.28 180) (fields_autoplaced yes)
+    (effects (font (size 1.27 1.27)) (justify right bottom)))
   (label "CAM_SCL" (at 88.9 83.82 0) (fields_autoplaced yes)
     (effects (font (size 1.27 1.27)) (justify left bottom)))
@@
   (label "UART7_RX" (at 88.9 96.52 0) (fields_autoplaced yes)
     (effects (font (size 1.27 1.27)) (justify left bottom)))
-  (no_connect (at 27.94 96.52))
+  (label "SPI2_MISO" (at 27.94 96.52 180) (fields_autoplaced yes)
+    (effects (font (size 1.27 1.27)) (justify right bottom)))
   (label "UART7_TX" (at 88.9 99.06 0) (fields_autoplaced yes)
     (effects (font (size 1.27 1.27)) (justify left bottom)))
@@
     (instances (project "head" (path "/a08b5940-33cf-5ae8-8123-d7cbee5060cd" (reference "#PWR014") (unit 1))))
   )
-  (no_connect (at 27.94 106.68))
+  (label "SPI2_CS0" (at 27.94 106.68 180) (fields_autoplaced yes)
+    (effects (font (size 1.27 1.27)) (justify right bottom)))
   (no_connect (at 88.9 109.22))
   (label "I2C8_SCL" (at 27.94 109.22 180) (fields_autoplaced yes)
@@
   (text "J11: LRC, BCLK, DIN, GAIN (open),\nSD (open: module's own pull-up), GND, Vin" (exclude_from_sim no) (at 467.36 358.14 0)
     (effects (font (size 1.27 1.27)) (justify left top)))
+  (rectangle (start 195 344) (end 395 400)
+    (stroke (width 0.2) (type dash)) (fill (type none)))
+  (text "SPI breakout" (exclude_from_sim no) (at 197 346 0)
+    (effects (font (size 2.0 2.0) bold) (justify left top)))
+  (text "SPI2 M1 for a future SPI device, untested. Wire pads on the bottom, under the module, along the top edge.\nCLK GPIO12 (CM4 31), MOSI GPIO13 (28), MISO GPIO22 (46), CS0 GPIO4 (54), INT GPIO6 (30), spare GPIO5 (34)" (exclude_from_sim no) (at 197 350 0)
+    (effects (font (size 1.27 1.27)) (justify left top)))
+  (symbol (lib_id "Connector_Generic:Conn_01x09") (at 238.76 375.92 0) (unit 1)
+    (exclude_from_sim no) (in_bom no) (on_board yes) (dnp no)
+    (property "Reference" "J13" (at 241.3 361.95 0)
+      (effects (font (size 1.27 1.27))))
+    (property "Value" "SPI pads" (at 248.92 375.92 0)
+      (effects (font (size 1.27 1.27))))
+    (property "Footprint" "DukkiHead:SolderPads_1x09_P2.54mm_SPI" (at 238.76 375.92 0)
+      (effects (font (size 1.27 1.27)) (hide yes)))
+    (property "Datasheet" "" (at 238.76 375.92 0)
+      (effects (font (size 1.27 1.27)) (hide yes)))
+    (property "Description" "" (at 238.76 375.92 0)
+      (effects (font (size 1.27 1.27)) (hide yes)))
+    (property "Note" "Bottom-side wire pads: G, 5V, 3V3, MO, MI, CK, CS, INT, IO" (at 238.76 375.92 0)
+      (effects (font (size 1.27 1.27)) (hide yes)))
+    (pin "1")
+    (pin "2")
+    (pin "3")
+    (pin "4")
+    (pin "5")
+    (pin "6")
+    (pin "7")
+    (pin "8")
+    (pin "9")
+    (instances (project "head" (path "/a08b5940-33cf-5ae8-8123-d7cbee5060cd" (reference "J13") (unit 1))))
+  )
+  (symbol (lib_id "power:GND") (at 233.68 365.76 270) (unit 1)
+    (exclude_from_sim no) (in_bom no) (on_board yes) (dnp no)
+    (property "Reference" "#PWR137" (at 233.68 360.68 90)
+      (effects (font (size 1.27 1.27)) (hide yes)))
+    (property "Value" "GND" (at 228.73 365.76 90)
+      (effects (font (size 1.27 1.27))))
+    (property "Footprint" "" (at 233.68 365.76 90)
+      (effects (font (size 1.27 1.27)) (hide yes)))
+    (property "Datasheet" "" (at 233.68 365.76 90)
+      (effects (font (size 1.27 1.27)) (hide yes)))
+    (property "Description" "" (at 233.68 365.76 90)
+      (effects (font (size 1.27 1.27)) (hide yes)))
+    (pin "1")
+    (instances (project "head" (path "/a08b5940-33cf-5ae8-8123-d7cbee5060cd" (reference "#PWR137") (unit 1))))
+  )
+  (symbol (lib_id "power:+5V") (at 233.68 368.3 90) (unit 1)
+    (exclude_from_sim no) (in_bom no) (on_board yes) (dnp no)
+    (property "Reference" "#PWR138" (at 233.68 363.22 90)
+      (effects (font (size 1.27 1.27)) (hide yes)))
+    (property "Value" "+5V" (at 228.73 368.3 90)
+      (effects (font (size 1.27 1.27))))
+    (property "Footprint" "" (at 233.68 368.3 90)
+      (effects (font (size 1.27 1.27)) (hide yes)))
+    (property "Datasheet" "" (at 233.68 368.3 90)
+      (effects (font (size 1.27 1.27)) (hide yes)))
+    (property "Description" "" (at 233.68 368.3 90)
+      (effects (font (size 1.27 1.27)) (hide yes)))
+    (pin "1")
+    (instances (project "head" (path "/a08b5940-33cf-5ae8-8123-d7cbee5060cd" (reference "#PWR138") (unit 1))))
+  )
+  (symbol (lib_id "power:+3V3") (at 233.68 370.84 90) (unit 1)
+    (exclude_from_sim no) (in_bom no) (on_board yes) (dnp no)
+    (property "Reference" "#PWR139" (at 233.68 365.76 90)
+      (effects (font (size 1.27 1.27)) (hide yes)))
+    (property "Value" "+3V3" (at 228.18 370.84 90)
+      (effects (font (size 1.27 1.27))))
+    (property "Footprint" "" (at 233.68 370.84 90)
+      (effects (font (size 1.27 1.27)) (hide yes)))
+    (property "Datasheet" "" (at 233.68 370.84 90)
+      (effects (font (size 1.27 1.27)) (hide yes)))
+    (property "Description" "" (at 233.68 370.84 90)
+      (effects (font (size 1.27 1.27)) (hide yes)))
+    (pin "1")
+    (instances (project "head" (path "/a08b5940-33cf-5ae8-8123-d7cbee5060cd" (reference "#PWR139") (unit 1))))
+  )
+  (label "SPI2_MOSI" (at 233.68 373.38 180) (fields_autoplaced yes)
+    (effects (font (size 1.27 1.27)) (justify right bottom)))
+  (label "SPI2_MISO" (at 233.68 375.92 180) (fields_autoplaced yes)
+    (effects (font (size 1.27 1.27)) (justify right bottom)))
+  (label "SPI2_CLK" (at 233.68 378.46 180) (fields_autoplaced yes)
+    (effects (font (size 1.27 1.27)) (justify right bottom)))
+  (label "SPI2_CS0" (at 233.68 381 180) (fields_autoplaced yes)
+    (effects (font (size 1.27 1.27)) (justify right bottom)))
+  (label "SPI_INT" (at 233.68 383.54 180) (fields_autoplaced yes)
+    (effects (font (size 1.27 1.27)) (justify right bottom)))
+  (label "SPI_IO" (at 233.68 386.08 180) (fields_autoplaced yes)
+    (effects (font (size 1.27 1.27)) (justify right bottom)))
+  (text "J13: 1 GND, 2 5V, 3 3V3, 4 MOSI, 5 MISO,\n6 CLK, 7 CS0, 8 INT, 9 spare GPIO" (exclude_from_sim no) (at 256.54 373.38 0)
+    (effects (font (size 1.27 1.27)) (justify left top)))
   (sheet_instances (path "/" (page "1")))

Commit message: Head carrier PCB rev B: pre-order review changes, USB download pads
- Buck input loop: C4 straight across U2's VIN and GND pins with ground
  vias beside them; boot cap and feedback divider at their pins.
- Input chain J1, TVS, C17 (47 uF 50 V electrolytic, C970679), then the
  ceramics; C3 dropped; fan parts moved down.
- 330R series resistors (R13, R14) in the link UART; J1 pins 3 and 4
  are now LINK_RX and LINK_TX.
- Bottom test pads: RST and BOOT (CM4 pins 92, 93), and USB D+, D-, G
  for the RK3576 download port (pins 105, 103) to flash in place.
  Pins checked against Radxa's CM4 schematic v1.20, sheets 8, 21, 22.
- J13 moved 2.5 mm clear of the module's M2.5 holes; J8 ends marked
  1 GND and 15 3V3.
- Top-layer keep-outs across the cut lines of JP1, JP3, JP4 and JP5
  (no tracks, vias or pour); crossing tracks rerouted.
- Tools: tidy and route_one_net treat locked copper of other nets as
  obstacles; tidy takes a board name, keeps socket ground tracks, never
  straightens through a pad, undangle runs one pass per process;
  route_one_net takes PCB, W, SRC and DST from the environment.
- DRC 0 violations with schematic parity; J9 pad 23 (ground, boxed in)
  unconnected, grounded inside the module. JLC package, PDFs and renders
  regenerated; design note sections 4 and 9.4.
Parts:
- added R13, R14: 330R, Resistor_SMD:R_0603_1608Metric, symbol Device:R
- added TP1: CM4_RESET, TestPoint:TestPoint_Pad_D1.5mm, symbol Connector:TestPoint
- added TP2: CM4_MASKROM, TestPoint:TestPoint_Pad_D1.5mm, symbol Connector:TestPoint
- added TP3, TP6: GND, TestPoint:TestPoint_Pad_D1.5mm, symbol Connector:TestPoint
- added TP4: USB_DN, TestPoint:TestPoint_Pad_D1.5mm, symbol Connector:TestPoint
- added TP5: USB_DP, TestPoint:TestPoint_Pad_D1.5mm, symbol Connector:TestPoint
- C17: renamed from C3; value 2.2u 50V -> 47u 50V; footprint Capacitor_SMD:C_0805_2012Metric -> Capacitor_SMD:CP_Elec_6.3x7.7; symbol Device:C -> Device:C_Polarized; LCSC C377773 -> C970679; MPN (none) -> RVT1H470M0607, 47 uF 50 V aluminium, 6.3 x 7.7 mm
Connections:
- net GND: now also TP3.1, TP6.1
- net UART7_RX: now also R13.1; no longer J1.3 (Pin_3)
- net UART7_TX: now also R14.1; no longer J1.4 (Pin_4)
- net USB_DN: now reaches J10.103 (USB2_N)
- net USB_DN: now also TP4.1
- net USB_DP: now reaches J10.105 (USB2_P)
- net USB_DP: now also TP5.1
- net CM4_RESET: now reaches J9.92 (RUN_PG)
- net CM4_RESET: now also TP1.1
- net CM4_MASKROM: now reaches J9.93 (nRPIBOOT)
- net CM4_MASKROM: now also TP2.1
- new net LINK_RX: J1.3 (Pin_3), R13.2
- new net LINK_TX: J1.4 (Pin_4), R14.2
- no-connect marks 128 -> 124
Other:
- note added: "330R in each UART7 line limits current into an unpowered CM4 from the bridge. TP1/TP2 (bottom): short to TP3 to reset; hold TP2 low through a reset for maskrom. TP4-TP6 (bottom): USB D-, D+, GND of the download port, for rkdeveloptool in maskrom"
- note added: "Link series resistors, test pads"

Commit message: Head carrier PCB: PWM pad for a possible mouth servo
- TP7, a bottom pad beside J9 on CM4 pin 37 (GPIO7, RK3576 GPIO1_C0,
  PWM0_CH0_M1), in case the mouth J288 is swapped for a hobby servo. The
  servo would run from its own buck module fed from J12's B+ and G, not
  the head's 5 V buck. PWM0 is separate from the fan's PWM1.
- Pin 48 (PWM1_CH0_M2) was tried first; on J9's inner row it is boxed in.
- Design note: J13 already gives spare GPIOs with 3V3 and GND (pads 8, 9
  and the SPI2 lines); a separate breakout under the module was tried and
  dropped (only a 130 mm, 11-via route).
- DRC 0 violations with schematic parity (J9 pad 23 as before); JLC
  package, PDFs and bottom render regenerated.
Parts:
- added TP7: SERVO_PWM, TestPoint:TestPoint_Pad_D1.5mm, symbol Connector:TestPoint
Connections:
- net SERVO_PWM: now reaches J9.37 (GPIO7)
- net SERVO_PWM: now also TP7.1
- no-connect marks 124 -> 123
Other:
- note added: "330R in each UART7 line limits current into an unpowered CM4 from the bridge. TP1/TP2 (bottom): short to TP3 to reset; hold TP2 low through a reset for maskrom. TP4-TP6 (bottom): USB D-, D+, GND of the download port, for rkdeveloptool in maskrom. TP7: GPIO7 / PWM0_CH0_M1 (pin 37) for a servo"
- note removed: "330R in each UART7 line limits current into an unpowered CM4 from the bridge. TP1/TP2 (bottom): short to TP3 to reset; hold TP2 low through a reset for maskrom. TP4-TP6 (bottom): USB D-, D+, GND of the download port, for rkdeveloptool in maskrom"
Changed lines of the file:
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@@
   (label "CAM_SDA" (at 27.94 83.82 180) (fields_autoplaced yes)
     (effects (font (size 1.27 1.27)) (justify right bottom)))
-  (no_connect (at 88.9 86.36))
+  (label "SERVO_PWM" (at 88.9 86.36 0) (fields_autoplaced yes)
+    (effects (font (size 1.27 1.27)) (justify left bottom)))
   (no_connect (at 27.94 86.36))
   (no_connect (at 88.9 88.9))
@@
   (text "Link series resistors, test pads" (exclude_from_sim no) (at 407 386 0)
     (effects (font (size 2.0 2.0) bold) (justify left top)))
-  (text "330R in each UART7 line limits current into an unpowered CM4 from the bridge. TP1/TP2 (bottom): short to TP3 to reset; hold TP2 low through a reset for maskrom.\nTP4-TP6 (bottom): USB D-, D+, GND of the download port, for rkdeveloptool in maskrom" (exclude_from_sim no) (at 407 390 0)
+  (text "330R in each UART7 line limits current into an unpowered CM4 from the bridge. TP1/TP2 (bottom): short to TP3 to reset; hold TP2 low through a reset for maskrom.\nTP4-TP6 (bottom): USB D-, D+, GND of the download port, for rkdeveloptool in maskrom. TP7: GPIO7 / PWM0_CH0_M1 (pin 37) for a servo" (exclude_from_sim no) (at 407 390 0)
     (effects (font (size 1.27 1.27)) (justify left top)))
   (symbol (lib_id "Device:R") (at 431.8 400.05 90) (unit 1)
@@
     (instances (project "head" (path "/a08b5940-33cf-5ae8-8123-d7cbee5060cd" (reference "#PWR141") (unit 1))))
   )
+  (symbol (lib_id "Connector:TestPoint") (at 558.8 410.21 0) (unit 1)
+    (exclude_from_sim no) (in_bom no) (on_board yes) (dnp no)
+    (property "Reference" "TP7" (at 558.8 405.13 0)
+      (effects (font (size 1.27 1.27))))
+    (property "Value" "SERVO_PWM" (at 558.8 415.29 0)
+      (effects (font (size 1.27 1.27))))
+    (property "Footprint" "TestPoint:TestPoint_Pad_D1.5mm" (at 558.8 410.21 0)
+      (effects (font (size 1.27 1.27)) (hide yes)))
+    (property "Datasheet" "" (at 558.8 410.21 0)
+      (effects (font (size 1.27 1.27)) (hide yes)))
+    (property "Description" "" (at 558.8 410.21 0)
+      (effects (font (size 1.27 1.27)) (hide yes)))
+    (pin "1")
+    (instances (project "head" (path "/a08b5940-33cf-5ae8-8123-d7cbee5060cd" (reference "TP7") (unit 1))))
+  )
+  (label "SERVO_PWM" (at 558.8 410.21 270) (fields_autoplaced yes)
+    (effects (font (size 1.27 1.27)) (justify right bottom)))
   (sheet_instances (path "/" (page "1")))
 )
